File: schematics/Switchboard.kicad_sch (KiCad schematic)
At the start: 4 parts

Commit message: commit
Parts:
- added K1: FINDER-34.51, Relay_THT:Relay_SPDT_Finder_34.51_Vertical, symbol Relay:FINDER-34.51
Connections:
- net at T1.4 (-VO), U1.14 (GND): now also J_RCsignal.2 (Pin_2)
- net at T1.3 (+VO), U1.19 (5V): now also K1.A1
- net at U1.23 (TOUCH3/HSPI_CS0/GPIO15): now also K1.14
- net at U1.28 (GPIO17): no longer J_RCsignal.2 (Pin_2)
- net at U1.38 (GND): now also K1.11; no longer J_RCsignal.1 (Pin_1)
- new net: J_RCsignal.1 (Pin_1), K1.A2
Other:
- moved on the sheet: J_230V, J_RCsignal, T1, U1
